File: PCB/Prayag's Macropad.kicad_pcb (KiCad board)
At the start: 2 copper layers, 100 x 71.4 mm, 29 parts, among them SW1 SW_Push, SW10 SW_Push, SW11 SW_Push, SW12 SW_Push, SW14 RotaryEncoder_Switch, SW2 SW_Push, SW3 SW_Push, SW4 SW_Push, SW5 SW_Push, SW6 SW_Push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

Commit message: review
Parts:
- removed C1: C, Capacitor_SMD:C_0805_2012Metric_Pad1.18x1.45mm_HandSolder
- removed R2: R, Resistor_SMD:R_0805_2012Metric_Pad1.20x1.40mm_HandSolder
Connections:
- U1 pad 4: Net-(U1-GPIO29/ADC3/A3) -> Net-(D1-DIN)
Routing:
- net Net-(U1-GPIO29/ADC3/A3): track 37.5 -> 0.00 mm
- net Net-(D1-DIN): track 9.67 -> 46.4 mm
- net +5V: track 64.0 -> 44.5 mm
- net GND: track 76.8 -> 74.8 mm
- net Row2: track 144.0 -> 142.9 mm
- net Col2: vias 2 -> 1
